File: fido2-lpc55.kicad_pcb (KiCad board)
At the start: 2 copper layers, 21.8 x 16.3 mm, 41 parts, among them J1 USB_A, J2 Conn_01x04, J3 Conn_01x05, T1 TLV742p, U1 LPC55S69JEV98K, U2 MTCH101, U3 SE050, Y1 XRCGB16M000FXN01R0

Commit message: NK3AN132
Parts:
- removed R5, R7: 4.7k, Resistor_SMD:R_0402_1005Metric
- removed R8: DNP, Resistor_SMD:R_0402_1005Metric
- added C5: 20pF, Capacitor_SMD:C_0402_1005Metric, F.Cu at (145.1, 91.3)
- C2: value 100n -> 100nF
- CY1: value 120pF -> 8pF
- R2: value 4.7k -> 1k
- U2: value MTCH101 -> TTP233D-HA6; footprint Package_TO_SOT_SMD:SOT-23-6 -> Package_TO_SOT_SMD:TSOT-23-6
- moved R3 1.02 mm to (145.2, 92.7)
- moved U2 0.40 mm to (148.2, 92.6)
Connections:
- R2 pad 2: Net-(R2-Pad2) -> Net-(C5-Pad1)
- U2 pad 1: Net-(R2-Pad2) -> /solo/Sheet5DDC9C58/SENSE1
- U2 pad 3: Net-(R5-Pad1) -> Net-(C5-Pad1)
- U2 pad 4: /solo/Sheet5DDC9C58/SENSE1 -> +3V3
- U2 pad 6: /solo/Sheet5DDC9C58/SENSE3 -> GNDREF
Routing:
- net GNDREF: track 145.9 -> 153.9 mm, vias 18 -> 20
- net Net-(C5-Pad1): track 0.00 -> 7.36 mm
- net Net-(R5-Pad1): track 4.83 -> 0.00 mm
- net /solo/Sheet5DDC9C58/SENSE1: track 6.87 -> 9.67 mm, vias 2 -> 3
- net Net-(R5-Pad2): track 2.31 -> 0.00 mm
- net /solo/Sheet5DDC9C58/SENSE3: track 1.75 -> 0.00 mm
- net Net-(R2-Pad2): track 1.42 -> 0.00 mm
- net +3V3: track 69.7 -> 70.5 mm
Other:
- board text added: "Nitrokey NK3AN 0622"
- board text removed: "Nitrokey NK3AN"
