File: solo.sch (KiCad schematic (older format))
At the start: 18 parts, among them J2 Conn_01x04, T1 TLV742p, U2 MTCH101

Commit message: NK3AN132
Parts:
- removed R5, R7: 4.7k, Resistor_SMD:R_0402_1005Metric, symbol Device:R
- removed R8: DNP, Resistor_SMD:R_0402_1005Metric, symbol Device:R
- removed U2: MTCH101, Package_TO_SOT_SMD:SOT-23-6, symbol fido2-lpc55-rescue:MTCH101-nk-fido2-solo-A-rescue
- added C5: 20pF, Capacitor_SMD:C_0402_1005Metric, symbol Device:C
- added U2: TTP233D-HA6, Package_TO_SOT_SMD:TSOT-23-6, symbol corelib:TTP233
- C2: value 100n -> 100nF
- CY1: value 120pF -> 8pF
- R2: value 4.7k -> 1k
Connections:
- wire segments 140 -> 145
- no-connect marks 3 -> 4
Other:
- moved on the sheet: R2
Changed lines of the file:
@@
 P 6250 5150
 F 0 "C2" H 6365 5196 50  0000 L CNN
-F 1 "100n" H 6365 5105 50  0000 L CNN
+F 1 "100nF" H 6365 5105 50  0000 L CNN
 F 2 "Capacitor_SMD:C_0402_1005Metric" H 6288 5000 50  0001 C CNN
 F 3 "~" H 6250 5150 50  0001 C CNN
@@
 	6400 4250 6700 4250
 $Comp
-L Device:R R5
-U 1 1 5DF7CDFF
-P 9000 1750
-F 0 "R5" H 9070 1796 50  0000 L CNN
-F 1 "4.7k" H 9070 1705 50  0000 L CNN
-F 2 "Resistor_SMD:R_0402_1005Metric" V 8930 1750 50  0001 C CNN
-F 3 "~" H 9000 1750 50  0001 C CNN
-F 4 "" H 9000 1750 50  0001 C CNN "Manufacturer"
-F 5 "+/- 1%" H 9000 1750 50  0001 C CNN "Description"
-F 6 "" H 9000 1750 50  0001 C CNN "MPN"
-F 7 "2" H 9000 1750 50  0001 C CNN "Pins"
-F 8 "0402" H 9000 1750 50  0001 C CNN "Package"
-	1    9000 1750
-	0    1    1    0
-$EndComp
-$Comp
-L fido2-lpc55-rescue:MTCH101-nk-fido2-solo-A-rescue U2
-U 1 1 5F3333B7
-P 9600 1650
-AR Path="/5F3333B7" Ref="U2"  Part="1"
-AR Path="/5DDFB633/5F3333B7" Ref="U2"  Part="1"
-F 0 "U2" H 9625 2037 60  0000 C CNN
-F 1 "MTCH101" H 9625 1931 60  0000 C CNN
-F 2 "Package_TO_SOT_SMD:SOT-23-6" H 9700 1400 60  0001 C CNN
-F 3 "" H 9700 1400 60  0001 C CNN
-	1    9600 1650
-	1    0    0    -1
-$EndComp
-$Comp
 L power:+3.3V #PWR0132
 U 1 1 5F3340BB
-P 10100 1650
-F 0 "#PWR0132" H 10100 1500 50  0001 C CNN
-F 1 "+3.3V" H 10115 1823 50  0000 C CNN
-F 2 "" H 10100 1650 50  0001 C CNN
-F 3 "" H 10100 1650 50  0001 C CNN
-	1    10100 1650
-	0    1    1    0
-$EndComp
-$Comp
-L power:GNDREF #PWR0133
-U 1 1 5F334592
-P 9150 1650
-F 0 "#PWR0133" H 9150 1400 50  0001 C CNN
-F 1 "GNDREF" H 9155 1477 50  0000 C CNN
-F 2 "" H 9150 1650 50  0001 C CNN
-F 3 "" H 9150 1650 50  0001 C CNN
-	1    9150 1650
-	0    1    1    0
+P 9850 1250
+F 0 "#PWR0132" H 9850 1100 50  0001 C CNN
+F 1 "+3.3V" H 9865 1423 50  0000 C CNN
+F 2 "" H 9850 1250 50  0001 C CNN
+F 3 "" H 9850 1250 50  0001 C CNN
+	1    9850 1250
+	1    0    0    -1
 $EndComp
 $Comp
 L Device:R R2
 U 1 1 5F339F25
-P 9150 1400
-F 0 "R2" H 9220 1446 50  0000 L CNN
-F 1 "4.7k" H 9220 1355 50  0000 L CNN
-F 2 "Resistor_SMD:R_0402_1005Metric" V 9080 1400 50  0001 C CNN
-F 3 "~" H 9150 1400 50  0001 C CNN
-F 4 "" H 9150 1400 50  0001 C CNN "Manufacturer"
-F 5 "+/- 1%" H 9150 1400 50  0001 C CNN "Description"
-F 6 "" H 9150 1400 50  0001 C CNN "MPN"
-F 7 "2" H 9150 1400 50  0001 C CNN "Pins"
-F 8 "0402" H 9150 1400 50  0001 C CNN "Package"
-	1    9150 1400
-	1    0    0    -1
-$EndComp
-Text Label 9150 1250 0    50   ~ 0
+P 8800 1450
+F 0 "R2" H 8870 1496 50  0000 L CNN
+F 1 "1k" H 8870 1405 50  0000 L CNN
+F 2 "Resistor_SMD:R_0402_1005Metric" V 8730 1450 50  0001 C CNN
+F 3 "~" H 8800 1450 50  0001 C CNN
+F 4 "" H 8800 1450 50  0001 C CNN "Manufacturer"
+F 5 "+/- 1%" H 8800 1450 50  0001 C CNN "Description"
+F 6 "" H 8800 1450 50  0001 C CNN "MPN"
+F 7 "2" H 8800 1450 50  0001 C CNN "Pins"
+F 8 "0402" H 8800 1450 50  0001 C CNN "Package"
+	1    8800 1450
+	1    0    0    -1
+$EndComp
+Text Label 8800 1300 0    50   ~ 0
 CAPT
 $Comp
@@
 	2300 4150 2700 4150
 $Comp
-L Device:R R7
-U 1 1 5FA4E5AE
-P 8650 1600
-F 0 "R7" H 8720 1646 50  0000 L CNN
-F 1 "4.7k" H 8720 1555 50  0000 L CNN
-F 2 "Resistor_SMD:R_0402_1005Metric" V 8580 1600 50  0001 C CNN
-F 3 "~" H 8650 1600 50  0001 C CNN
-F 4 "" H 8650 1600 50  0001 C CNN "Manufacturer"
-F 5 "+/- 1%" H 8650 1600 50  0001 C CNN "Description"
-F 6 "" H 8650 1600 50  0001 C CNN "MPN"
-F 7 "2" H 8650 1600 50  0001 C CNN "Pins"
-F 8 "0402" H 8650 1600 50  0001 C CNN "Package"
-	1    8650 1600
-	-1   0    0    1
-$EndComp
-$Comp
-L Device:R R8
-U 1 1 5FA4EB11
-P 8650 1900
-F 0 "R8" H 8720 1946 50  0000 L CNN
-F 1 "DNP" H 8720 1855 50  0000 L CNN
-F 2 "Resistor_SMD:R_0402_1005Metric" V 8580 1900 50  0001 C CNN
-F 3 "~" H 8650 1900 50  0001 C CNN
-F 4 "" H 8650 1900 50  0001 C CNN "Manufacturer"
-F 5 "+/- 1%" H 8650 1900 50  0001 C CNN "Description"
-F 6 "" H 8650 1900 50  0001 C CNN "MPN"
-F 7 "2" H 8650 1900 50  0001 C CNN "Pins"
-F 8 "0402" H 8650 1900 50  0001 C CNN "Package"
-	1    8650 1900
-	-1   0    0    1
-$EndComp
-$Comp
-L power:+3.3V #PWR012
-U 1 1 5FA4ED2E
-P 8650 1450
-F 0 "#PWR012" H 8650 1300 50  0001 C CNN
-F 1 "+3.3V" H 8665 1623 50  0000 C CNN
-F 2 "" H 8650 1450 50  0001 C CNN
-F 3 "" H 8650 1450 50  0001 C CNN
-	1    8650 1450
-	1    0    0    -1
-$EndComp
-Wire Wire Line
-	8650 1750 8850 1750
-Connection ~ 8650 1750
-$Comp
-L power:GNDREF #PWR013
-U 1 1 5FA55230
-P 8650 2050
-F 0 "#PWR013" H 8650 1800 50  0001 C CNN
-F 1 "GNDREF" H 8655 1877 50  0000 C CNN
-F 2 "" H 8650 2050 50  0001 C CNN
-F 3 "" H 8650 2050 50  0001 C CNN
-	1    8650 2050
-	1    0    0    -1
-$EndComp
-$Comp
 L Device:C CY1
 U 1 1 6056EDA3
 P 2700 4000
 F 0 "CY1" H 2815 4046 50  0000 L CNN
-F 1 "120pF" H 2815 3955 50  0000 L CNN
+F 1 "8pF" H 2815 3955 50  0000 L CNN
 F 2 "Capacitor_SMD:C_0402_1005Metric" H 2738 3850 50  0001 C CNN
 F 3 "~" H 2700 4000 50  0001 C CNN
@@
 Wire Wire Line
 	2700 4150 3050 4150
+$Comp
+L corelib:TTP233 U2
+U 1 1 62BC05F5
+P 9800 1850
+F 0 "U2" H 9500 1550 50  0000 L CNN
+F 1 "TTP233D-HA6" H 9450 2300 50  0000 L CNN
+F 2 "Package_TO_SOT_SMD:TSOT-23-6" H 9800 1850 50  0001 C CNN
+F 3 "" H 9800 1850 50  0001 C CNN
+	1    9800 1850
+	1    0    0    -1
+$EndComp
+Wire Wire Line
+	9850 1250 9850 1350
+NoConn ~ 10100 1550
+Wire Wire Line
+	9400 1900 9400 2150
+Wire Wire Line
+	9400 2150 9900 2150
+$Comp
+L power:GNDREF #PWR013
+U 1 1 62BEE521
+P 9900 2150
+F 0 "#PWR013" H 9900 1900 50  0001 C CNN
+F 1 "GNDREF" H 9905 1977 50  0000 C CNN
+F 2 "" H 9900 2150 50  0001 C CNN
+F 3 "" H 9900 2150 50  0001 C CNN
+	1    9900 2150
+	1    0    0    -1
+$EndComp
+Connection ~ 9900 2150
+$Comp
+L power:+3.3V #PWR012
+U 1 1 62BEEA89
+P 9400 1800
+F 0 "#PWR012" H 9400 1650 50  0001 C CNN
+F 1 "+3.3V" H 9415 1973 50  0000 C CNN
+F 2 "" H 9400 1800 50  0001 C CNN
+F 3 "" H 9400 1800 50  0001 C CNN
+	1    9400 1800
+	0    -1   -1   0
+$EndComp
+$Comp
+L Device:C C5
+U 1 1 62BEF6D4
+P 8800 1750
+F 0 "C5" H 8915 1796 50  0000 L CNN
+F 1 "20pF" H 8915 1705 50  0000 L CNN
+F 2 "Capacitor_SMD:C_0402_1005Metric" H 8838 1600 50  0001 C CNN
+F 3 "~" H 8800 1750 50  0001 C CNN
+F 4 "" H 8800 1750 50  0001 C CNN "Manufacturer"
+F 5 "" H 8800 1750 50  0001 C CNN "Description"
+F 6 "" H 8800 1750 50  0001 C CNN "MPN"
+F 7 "2" H 8800 1750 50  0001 C CNN "Pins"
+F 8 "0402" H 8800 1750 50  0001 C CNN "Package"
+	1    8800 1750
+	1    0    0    -1
+$EndComp
+Wire Wire Line
+	9400 1600 8800 1600
+Connection ~ 8800 1600
+Wire Wire Line
+	9400 2150 8800 2150
+Wire Wire Line
+	8800 2150 8800 1900
+Connection ~ 9400 2150
 $EndSCHEMATC
